Commit message: [BugFix] update xarco file

File: models/rotors_description/urdf/multirotor_base.xacro (robot description, xacro)
@@ -92,5 +92,5 @@
       </visual>
       <collision>
-        <origin xyz="0 0 0" rpy="0 0 0" />
+        <origin xyz="0 0 0.61" rpy="0 0 0" />
         <geometry>
          <cylinder length="1.0" radius="0.005" /> <!-- [m] -->
